File: hardware/ablerex-rs1000-tester/analog_filter.kicad_sch (KiCad schematic)
At the start: 86 parts, among them U16 TL074, U17 TL072, U18 TL074, U9 LM339

Commit message: progress on schematic
Parts:
- added C78: DNP (1n), symbol Device:C_Small
- added C81: DNP, symbol Device:C_Small
- added C82, C83, C84, C85, C86, C88, C90, C92: 100n, symbol Device:C_Small
- added C87, C89, C91, C93, C94, C95: 1n, symbol Device:C_Small
- added D27, D30, D31, D32, D33, D34, D35: BAV99, Package_TO_SOT_SMD:SOT-23, symbol Diode:BAV99
- added D28, D29: 1N4148WS, Diode_SMD:D_SOD-323, symbol Diode:1N4148WS
- added R151, R152, R155, R156, R157, R159, R160, R162, R163, R164, R165, R167, R168, R169, R172, R175: 10K, symbol Device:R_Small
- added R153, R154: 25K5, symbol Device:R_Small
- added R158, R166, R171, R174: 330R, symbol Device:R_Small
- added R161, R170, R173, R176, R177, R180, R183: 4K99, symbol Device:R_Small
- added R178, R181, R184: 1K, symbol Device:R_Small
- added R179, R182, R185: 0R, symbol Device:R_Small
- added U19, U20: TL074, symbol Amplifier_Operational:TL074
Connections:
- net +1.65Vad: now also R176.1, U20.13 (-)
- net +12VA: now also C82.1, C85.1, U19.4 (V+), U20.4 (V+)
- net +3.3Vad: now also D27.2 (A), D30.2 (A), D31.2 (A), D32.2 (A), D33.2 (A), D34.2 (A), D35.2 (A), R156.2, R177.2, R180.2, R183.2
- net -12VA: now also C83.2, C86.2, U19.11 (V-), U20.11 (V-)
- net ADgnd: now also C82.2, C83.1, C84.2, C85.2, C86.1, C88.2, C90.2, C92.2, C93.2, C94.2, C95.2, D27.1 (K), D30.1 (K), D31.1 (K), D32.1 (K), D33.1 (K), D34.1 (K), D35.1 (K), R153.1, R168.1, R179.1, R182.1, R185.1, U19.10 (+), U19.12 (+), U20.12 (+)
- new net: D28.2 (A), D29.1 (K), U19.8
- new net: D29.2 (A), R160.2, R161.1
- new net: R169.2, R170.1, U20.6 (-)
- new net: R170.2, R171.1, U20.7
- new net: R172.2, R173.1, U20.9 (-)
- new net: C81.1, R157.2, R158.1, U19.7
- new net: D28.1 (K), R159.2, R160.1, U19.9 (-)
- new net: R161.2, R162.1, R163.2, U19.13 (-)
- new net: R155.2, R156.1, U19.5 (+)
- new net: C81.2, R157.1, U19.6 (-)
- new net: R165.2, R166.1, U20.1
- new net: R167.2, R168.2, U20.3 (+)
- new net: R175.2, R176.2, U20.10 (+)
- new net: R173.2, R174.1, U20.8
- new net: R154.2, R155.1, R159.1, R163.1, U19.1
- new net: R151.2, R154.1, U19.2 (-)
- new net: R152.2, R153.2, U19.3 (+)
- new net: R164.2, R165.1, U20.2 (-)
- new net A/D_Charger C: C88.1, D30.3 (K), R166.2
- new net A/D_Input relay V: C92.1, D32.3 (K), R174.2
- new net A/D_Inverter Output C: C84.1, D27.3 (K), R158.2
- new net A/D_Output Relay V: C90.1, D31.3 (K), R171.2
- new net A/D_Temperature1: C93.1, D33.3 (K), R178.2
- new net A/D_Temperature2: C94.1, D34.3 (K), R181.2
- new net A/D_UPS KVA: C95.1, D35.3 (K), R184.2
- new net Charger Current Sensor_+: C87.2, R167.1, U20.5 (+)
- new net Charger Current Sensor_-: C87.1, R164.1
- new net Input relay V_+: C91.2, R175.1
- new net Input relay V_-: C91.1, R172.1
- new net Inverter Output C: R162.2, U19.14
- new net Inverter Output C_+: C78.2, R152.1
- new net Inverter Output C_-: C78.1, R151.1
- new net Inverter Output V_-: C89.2
- new net Output Relay V_+: C89.1, R169.1
- new net Temperature Sensor1_+: R177.1, R178.1
- new net Temperature Sensor1_-: R179.2
- new net Temperature Sensor2_+: R180.1, R181.1
- new net Temperature Sensor2_-: R182.2
- new net UPS KVA select_+: R183.1, R184.1
- new net UPS KVA select_-: R185.2
- no-connect marks 0 -> 1

Commit message: Completed the schematic, checked until 40th pin of the MCU
Parts:
- C67: value 1n -> DNP (1n)
Connections:
- net +1.65Vad: no longer R128.1
- net ADgnd: now also R128.1
- net A/D_DCBUS(+): no longer C75.1, D25.3 (K), R145.2
- net Charger Current Sensor_+: no longer U20.5 (+)
- net CommInvRelay: now also U20.5 (+)
- net Input V_+: no longer C58.2, R116.1
- net Input V_-: no longer C58.1, R114.1
- net Inverter Output V_-: now also C58.2, R116.1
- new net A/D_DCBUS(-): C75.1, D25.3 (K), R145.2
- new net Inverter Output V_+: C58.1, R114.1
Changed lines of the file:
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@@
 	)
 	(junction
+		(at 73.66 247.65)
+		(diameter 0)
+		(color 0 0 0 0)
+	)
+	(junction
 		(at 62.23 92.71)
 		(diameter 0)
@@
 	(wire
 		(pts
-			(xy 54.61 247.65) (xy 57.15 247.65)
+			(xy 54.61 247.65) (xy 73.66 247.65)
 		)
 		(stroke
@@
 	)
 	(rectangle
-		(start 15.24 80.01)
+		(start 8.89 80.01)
 		(end 115.57 123.19)
 		(stroke
@@
 		)
 	)
-	(global_label "Charger Current Sensor_+"
+	(global_label "CommInvRelay"
 		(shape input)
 		(at 363.22 346.71 180)
@@
 		)
 		(property "Intersheetrefs" "${INTERSHEET_REFS}"
-			(at 335.0165 346.71 0)
+			(at 346.5674 346.71 0)
 			(effects
 				(font
@@
 		)
 	)
-	(global_label "Input V_-"
+	(global_label "Inverter Output V_+"
 		(shape input)
 		(at 31.75 92.71 180)
@@
 		)
 		(property "Intersheetrefs" "${INTERSHEET_REFS}"
-			(at 19.3911 92.71 0)
+			(at 9.7754 92.71 0)
 			(effects
 				(font
@@
 		)
 	)
-	(global_label "Input V_+"
+	(global_label "Inverter Output V_-"
 		(shape input)
 		(at 31.75 105.41 180)
@@
 		)
 		(property "Intersheetrefs" "${INTERSHEET_REFS}"
-			(at 19.3911 105.41 0)
+			(at 9.7754 105.41 0)
 			(effects
 				(font
@@
 		)
 	)
-	(global_label "A{slash}D_DCBUS(+)"
+	(global_label "A{slash}D_DCBUS(-)"
 		(shape input)
 		(at 375.92 31.75 0)
@@
 	)
 	(symbol
-		(lib_id "power:+1V5")
-		(at 57.15 247.65 270)
-		(unit 1)
-		(exclude_from_sim no)
-		(in_bom yes)
-		(on_board yes)
-		(dnp no)
-		(property "Reference" "#PWR0138"
-			(at 53.34 247.65 0)
-			(effects
-				(font
-					(size 1.27 1.27)
-				)
-				(hide yes)
-			)
-		)
-		(property "Value" "+1.65Vad"
-			(at 65.024 247.65 90)
-			(effects
-				(font
-					(size 1.27 1.27)
-				)
-			)
-		)
-		(property "Footprint" ""
-			(at 57.15 247.65 0)
-			(effects
-				(font
-					(size 1.27 1.27)
-				)
-				(hide yes)
-			)
-		)
-		(property "Datasheet" ""
-			(at 57.15 247.65 0)
-			(effects
-				(font
-					(size 1.27 1.27)
-				)
-				(hide yes)
-			)
-		)
-		(property "Description" "Power symbol creates a global label with name \"+1V5\""
-			(at 57.15 247.65 0)
-			(effects
-				(font
-					(size 1.27 1.27)
-				)
-				(hide yes)
-			)
-		)
-		(pin "1"
-		)
-		(instances
-			(project "ablerex-rs1000-tester"
-				(path "/4f9ff883-ac43-4f43-936a-c87cd548c592/5078029d-fd39-43c4-9e36-dc2747e0beb1"
-					(reference "#PWR0138")
-					(unit 1)
-				)
-			)
-		)
-	)
-	(symbol
 		(lib_id "Device:R_Small")
 		(at 52.07 160.02 270)
@@
 		(on_board yes)
 		(dnp no)
-		(fields_autoplaced yes)
 		(property "Reference" "C67"
-			(at 35.56 232.4162 0)
+			(at 24.384 232.664 0)
 			(effects
 				(font
@@
 			)
 		)
-		(property "Value" "1n"
-			(at 35.56 234.9562 0)
+		(property "Value" "DNP (1n)"
+			(at 22.352 235.458 0)
 			(effects
 				(font

Commit message: checked all the schematics
Other:
- moved on the sheet: C91, C92, C93, D32, D33, R172, R173, R174, R175, R176, R177, R178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
