File: hardware/ablerex-rs1000-tester/comm_and_power.kicad_sch (KiCad schematic)
At the start: 72 parts, among them J10 Conn_01x04, J11 Conn_02x13_Odd_Even, J9 Conn_01x05, Q1 MMBTA42, Q2 MMBT5551L, Q4 MMBTA42, T1 Transformer_1P_SS, U10 PC817, U11 PC817, U12 AMS1117-3.3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

Commit message: checked all the schematics
Connections:
- net Power_ON renamed I_UC3845(POWER) Power ON
Changed lines of the file:
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@@
+	(wire
+		(pts
+			(xy 19.05 177.8) (xy 19.05 179.07)
+		)
+		(stroke
+			(width 0)
+			(type default)
+		)
+	)
 	(wire
 		(pts
@@
 	(wire
 		(pts
-			(xy 27.94 176.53) (xy 30.48 176.53)
-		)
-		(stroke
-			(width 0)
-			(type default)
-		)
-	)
-	(wire
-		(pts
 			(xy 223.52 133.35) (xy 226.06 133.35)
 		)
@@
 	(wire
 		(pts
+			(xy 19.05 179.07) (xy 29.21 179.07)
+		)
+		(stroke
+			(width 0)
+			(type default)
+		)
+	)
+	(wire
+		(pts
 			(xy 57.15 30.48) (xy 57.15 33.02)
 		)
@@
 	(wire
 		(pts
+			(xy 29.21 176.53) (xy 30.48 176.53)
+		)
+		(stroke
+			(width 0)
+			(type default)
+		)
+	)
+	(wire
+		(pts
 			(xy 248.92 55.88) (xy 246.38 55.88)
 		)
@@
 		(pts
 			(xy 226.06 140.97) (xy 226.06 133.35)
+		)
+		(stroke
+			(width 0)
+			(type default)
+		)
+	)
+	(wire
+		(pts
+			(xy 29.21 179.07) (xy 29.21 176.53)
 		)
 		(stroke
@@
 		)
 	)
-	(global_label "Power_ON"
-		(shape input)
-		(at 27.94 176.53 180)
-		(fields_autoplaced yes)
-		(effects
-			(font
-				(size 1.27 1.27)
-			)
-			(justify right)
-		)
-		(property "Intersheetrefs" "${INTERSHEET_REFS}"
-			(at 15.7019 176.53 0)
-			(effects
-				(font
-					(size 1.27 1.27)
-				)
-				(justify right)
-				(hide yes)
-			)
+	(global_label "I_UC3845(POWER) Power ON"
+		(shape input)
+		(at 19.05 177.8 90)
+		(fields_autoplaced yes)
+		(effects
+			(font
+				(size 1.27 1.27)
+			)
+			(justify left)
+		)
+		(property "Intersheetrefs" "${INTERSHEET_REFS}"
+			(at 19.05 147.4191 90)
+			(effects
+				(font
+					(size 1.27 1.27)
+				)
+				(justify left)
+				(hide yes)
+			)
