File: hardware/ablerex-rs1000-tester/level-shifter.kicad_sch (KiCad schematic)
At the start: 30 parts, among them U1 ULN2003A, U2 74HC14, U3 25LCxxx, U4 74HCT240, U5 74HCT240

Commit message: checked all the schematics
Parts:
- added C97: 100n, symbol Device:C_Small
Connections:
- net +3.3VA: now also C97.1
- net AGND: now also U4.11 (2A3), U4.6 (1A2), U4.8 (1A3), U5.11 (2A3), U5.15 (2A1), C97.2; no longer U4.12 (1Y3), U4.14 (1Y2), U4.9 (2Y3), U5.5 (2Y1), U5.9 (2Y3)
- net Boost Charge Control: now also U5.3 (2Y0); no longer U5.17 (2A0)
- net Boost Charge Control(CPU): now also U5.17 (2A0); no longer U5.3 (2Y0)
- net Boost Control PWM 1: now also U4.7 (2Y2); no longer U4.13 (2A2)
- net Boost Control PWM1(CPU): now also U4.13 (2A2); no longer U4.7 (2Y2)
- net Boost Control PWM2: now also U4.5 (2Y1); no longer U4.15 (2A1)
- net Boost Control PWM2(CPU): now also U4.15 (2A1); no longer U4.5 (2Y1)
- net Charger Shutdown: now also U5.7 (2Y2); no longer U5.13 (2A2)
- net Charger Shutdown(CPU): now also U5.13 (2A2); no longer U5.7 (2Y2)
- net Input Current Protect: now also U2.9; no longer U2.11
- net Inv_Protect: now also C19.1, U2.1
- net Inverter Down Arm: now also U4.16 (1Y1); no longer U4.4 (1A1)
- net Inverter Down Arm(CPU): now also U4.4 (1A1); no longer U4.16 (1Y1)
- net Inverter Up Arm: now also U4.18 (1Y0); no longer U4.2 (1A0)
- net Inverter Up Arm(CPU): now also U4.2 (1A0); no longer U4.18 (1Y0)
- net O_Control FAN: now also U5.18 (1Y0); no longer U5.2 (1A0)
- net O_Control FAN(CPU): now also U5.2 (1A0); no longer U5.18 (1Y0)
- net O_SimSCITX: now also U5.12 (1Y3); no longer U5.8 (1A3)
- net O_TurboCurrent_Mode: now also U5.16 (1Y1); no longer U5.4 (1A1)
- net O_TurboCurrent_Mode(CPU): now also U5.4 (1A1); no longer U5.16 (1Y1)
- net Ouput Current Protect: now also U2.11; no longer U2.9
- net PFC Control: now also U4.3 (2Y0); no longer U4.17 (2A0)
- net PFC Control(CPU): now also U4.17 (2A0); no longer U4.3 (2Y0)
- net SCITXD(DSP): now also U5.6 (1A2); no longer U5.14 (1Y2)
- net SCITXD_inv: now also U5.14 (1Y2); no longer U5.6 (1A2)
- net TMS: now also U5.8 (1A3); no longer U5.12 (1Y3)
- net Enable_BufferIC: now reaches R23.1, U2.5
- net at U2.8: now also U1.6 (I6); no longer U1.5 (I5)
- net PFC_Protect: now reaches C18.1, U2.3
- net at U2.10: now also U1.5 (I5); no longer U1.6 (I6)
- no-connect marks 7 -> 8
Other:
- moved on the sheet: C18, C19, C20, C21, R13, R14, R15, R16, R17, R18, R19, R20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
