File: hardware/ablerex-rs1000-tester/protector.kicad_sch (KiCad schematic)
At the start: 29 parts, among them U9 LM339

Commit message: checked all the schematics
Connections:
- net at R63.2: now also U9.7 (+); no longer U9.6 (-)
- net at R64.1, R66.2: now also U9.6 (-); no longer U9.7 (+)
Changed lines of the file:
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@@
 		(lib_id "Comparator:LM339")
 		(at 129.54 86.36 0)
-		(mirror x)
 		(unit 2)
 		(exclude_from_sim no)
@@
 		(dnp no)
 		(property "Reference" "U9"
-			(at 133.858 82.804 0)
+			(at 133.858 89.916 0)
 			(effects
 				(font
@@
 		)
 		(property "Value" "LM339"
-			(at 135.636 88.9 0)
+			(at 135.636 83.82 0)
 			(effects
 				(font
@@
 		)
 		(property "Footprint" ""
-			(at 128.27 88.9 0)
+			(at 128.27 83.82 0)
 			(effects
 				(font
@@
 		)
 		(property "Datasheet" "https://www.st.com/resource/en/datasheet/lm139.pdf"
-			(at 130.81 91.44 0)
+			(at 130.81 81.28 0)
 			(effects
 				(font
